File: video_signal_generation/video_signal_generation.kicad_sch (KiCad schematic)
At the start: 26 parts, among them U1 74LS123, U2 TL072

Commit message: update schematic
Parts:
- removed BT1, BT2: 9V, symbol Device:Battery
- added J? (x3): Conn_01x01_Male, symbol Connector:Conn_01x01_Male
- added JP1: LOAD, symbol Jumper:Jumper_2_Open
- added R22: 1K, symbol Device:R
- D1, D2, D3: value D -> 1N4148
- U2: value TL072 -> MAX457
Connections:
- net GND: now also J?.1 (Pin_1)
- net OUTPUT: now reaches D1.1 (K), D2.2 (A), R7.2, TP4.1, U2.7
- net OUTPUT: now also JP1.1 (A); no longer R1000.1
- net -5VA: now reaches C12.2, U2.4 (V-)
- net -5VA: now also J?.1 (Pin_1)
- net at TP2.1, U1.11 (Clr): now also A1.14 (D11); no longer A1.13 (D10)
- net at C2.1, U1.7 (RCext): now also R22.2; no longer R2.2
- net +9V renamed +5VA
- net +5VA: now also J?.1 (Pin_1); no longer A1.30 (VIN)
- new net: JP1.2 (B), R1000.1
- new net: R2.2, R22.1
- no-connect marks 27 -> 28
Other:
- note added: "-0.3 V peak"
- note added: "adjust to 0.7 V peak"
- note added: "protection diodes"
- note added: "test load"
- note removed: "Monitor"
- moved on the sheet: R2, TP2
